File: firmware/ESPCord/ESPCord.kicad_sch (KiCad schematic)
At the start: 5 parts, among them J1 USB_C_Receptacle, K1 SRD-03VDC-SL-C, U1 ESP32-C3

Commit message: added the pcb, and now time to work on the Zine along with programming
Parts:
- added C1, C2: 10uF_0805_16V_lowESR, PCM_4ms_Capacitor:C_0805, symbol PCM_4ms_Capacitor:10uF_0805_16V_lowESR
- added U2: AMS1117-3_3_C347222, PCM_Package_TO_SOT_SMD_AKL:SOT-223-5, symbol JLCImport:AMS1117-3_3_C347222
Connections:
- net +3.3V: now also C2.1, U2.2 (VOUT(TAB))
- net 5V: now also K1.2, K1.5, C1.2, U2.3 (VIN); no longer K1.3
- net GPIO10: now reaches U1.16 (GPIO10)
- net GPIO10: now also K1.1
- net D-: now reaches J1.A7 (D-), J1.B7 (D-), U1.25 (GPIO18)
- net D+: now reaches J1.A6 (D+), J1.B6 (D+), U1.26 (GPIO19)
- net GND: now reaches J1.GND, R3.2, R4.2
- net GND: now also J1.S (SHIELD), K1.4, C1.1, C2.2, U2.1 (ADJ(GND))
Other:
- moved on the sheet: J1, K1, R3, R4
